Commit message: Update: STM32 Nucleo -> STM32F4, SLAM parameters optimized for map drift

File: src/my_robot_description/urdf/my_robot.urdf.xacro (robot description, xacro)
@@ -48,8 +48,9 @@
   </link>
   <!-- base_footprint -> base_link joint -->
+  <!-- base_footprint z=0 (yer seviyesi), base_link z=wheel_radius yukarıda -->
   <joint name="base_joint" type="fixed">
     <parent link="base_footprint"/>
     <child link="base_link"/>
-    <origin xyz="0 0 0" rpy="0 0 0"/>
+    <origin xyz="0 0 ${wheel_radius}" rpy="0 0 0"/>
   </joint>
   <!-- LIDAR -->

Commit message: Arduino firmware kodları eklendi
- ROSArduinoBridge firmware dosyaları eklendi (firmware klasörü)
- Motor driver (BTS7960), encoder, PID kontrol desteği
- Servo, buzzer, emergency button, DFPlayer Mini desteği
- Firmware README.md eklendi (kurulum ve kullanım rehberi)
- Tüm Arduino kodları tam ve çalışır durumda

File: src/my_robot_description/urdf/my_robot.urdf.xacro (robot description, xacro)
@@ -64,11 +64,11 @@
   </joint>
   <link name="laser_link">
-    <visual>
+      <visual>
       <origin xyz="0 0 0" rpy="0 0 0"/>
-      <geometry>
+        <geometry>
         <cylinder radius="${laser_radius}" length="${laser_length}"/>
-      </geometry>
+        </geometry>
       <material name="black"/>
-    </visual>
+      </visual>
     <collision>
       <origin xyz="0 0 0" rpy="0 0 0"/>
@@ -95,10 +95,10 @@
   </joint>
   <link name="left_wheel">
-    <collision>
+      <collision>
       <origin xyz="0 0 0" rpy="${PI/2} 0 0"/>
-      <geometry>
+        <geometry>
         <cylinder length="${wheel_len}" radius="${wheel_radius}"/>
-      </geometry>
-    </collision>
+        </geometry>
+      </collision>
     <visual>
       <origin xyz="0 0 0" rpy="${PI/2} 0 0"/>
@@ -108,21 +108,21 @@
       <material name="black"/>
     </visual>
-    <inertial>
-      <mass value="1.0"/>
-      <origin xyz="0 0 0"/>
+      <inertial>
+        <mass value="1.0"/>
+        <origin xyz="0 0 0"/>
       <inertia
         ixx="0.01" ixy="0" ixz="0"
         iyy="0.01" iyz="0"
         izz="0.01"/>
-    </inertial>
-  </link>
+      </inertial>
+    </link>
   <!-- Sağ Teker -->
   <joint name="right_wheel_joint" type="continuous">
-    <parent link="base_link"/>
+      <parent link="base_link"/>
     <child link="right_wheel"/>
     <origin xyz="0 -${base_width/2} 0" rpy="0 0 0"/>
-    <axis xyz="0 1 0"/>
+      <axis xyz="0 1 0"/>
     <dynamics damping="0.2"/>
-  </joint>
+    </joint>
   <link name="right_wheel">
     <collision>
