Commit message: Arduino haberleşme uyumluluğu ve test planı eklendi
- Arduino haberleşme protokolü detaylı kontrol edildi ve düzeltildi
- Motor komut hesaplaması Arduino PID_RATE ile uyumlu hale getirildi
- Baud rate ve port eşleşmeleri kontrol edildi ve düzeltildi
- ROS2 Control device parametresi launch'tan geçirilebilir hale getirildi
- arduino_bridge.py ve ROS2 Control çakışması uyarıları eklendi
- Tüm launch dosyalarına kritik uyarılar eklendi
- KURULUM_REHBERI.md güncellendi (donanım/yazılım kurulumu)
- TEST_PLANI.md eklendi (7 adımlı test planı)
- URDF wheel_radius Teknofest-AGV ile uyumlu hale getirildi
- YAML format hataları düzeltildi
- Odometry topic remapping eklendi

File: src/my_robot_description/ros2_control/my_robot.ros2_control.xacro (robot description, xacro)
@@ -3,5 +3,5 @@
   <!-- ROS2 Control hardware interface for Arduino -->
   <!-- Teknofest-AGV değerleriyle güncellendi (Raspberry Pi 5 + ROS2 Jazzy) -->
-  <xacro:macro name="my_robot_hardware" params="name">
+  <xacro:macro name="my_robot_hardware" params="name device:=/dev/ttyUSB0">
     <ros2_control name="${name}" type="system">
       <hardware>
@@ -10,5 +10,5 @@
         <param name="right_wheel_name">right_wheel_joint</param>
         <param name="loop_rate">40</param>
-        <param name="device">/dev/ttyUSB0</param>
+        <param name="device">${device}</param>
         <param name="baud_rate">57600</param>
         <param name="timeout_ms">1000</param>

File: src/my_robot_description/urdf/my_robot.urdf.xacro (robot description, xacro)
@@ -7,7 +7,9 @@
 - Differential drive with caster wheel
 - LIDAR mounted on top
-NOT: ros2_control entegrasyonu YOK (Micro-ROS kullanıyoruz)
+NOT: ROS2 Control entegrasyonu VAR (Arduino Mega ile haberleşme)
 -->
 <robot name="my_robot" xmlns:xacro="http://www.ros.org/wiki/xacro">
+  <!-- Xacro argümanları (launch dosyasından geçirilir) -->
+  <xacro:arg name="device" default="/dev/ttyUSB0" />
   <!-- Import materials -->
   <xacro:include filename="$(find my_robot_description)/urdf/my_robot.materials.xacro" />
@@ -20,5 +22,5 @@
   <xacro:property name="base_height" value="0.24" />
   <xacro:property name="wheel_len" value="0.030" />
-  <xacro:property name="wheel_radius" value="0.055" />
+  <xacro:property name="wheel_radius" value="0.055" />  <!-- Teknofest-AGV değeri (URDF fiziksel görünüm için) -->
   <xacro:property name="caster_wheel_radius" value="0.055" />
   <xacro:property name="axle_offset" value="0.10" />
@@ -180,4 +182,5 @@
   </link>
   <!-- ROS2 Control Hardware Interface -->
-  <xacro:my_robot_hardware name="MyRobotHardware"/>
+  <!-- device parametresi launch dosyasından geçirilir, varsayılan: /dev/ttyUSB0 -->
+  <xacro:my_robot_hardware name="MyRobotHardware" device="${device}"/>
 </robot>
